File: hw/subbat.sch (KiCad schematic (older format))
At the start: 154 parts, among them J1 Conn_01x02_Female, J10 USB_Ax2, J11 Conn_01x02_Female, J2 Barrel_Jack, J3 USB_Ax2, J4 USB_Ax2, J5 Conn_01x02_Female, J6 Conn_WallSocket, J7 USB_B_Micro, J8 USB_Ax2, J9 USB_Ax2, K1 953-1C-5DG-1, P1 Conn_WallPlug, P2 CONN_01X06, P3 CONN_01X06, P4 CONN_01X06, Q1 DMP3007SCG, Q2 2N7002, Q3 2N7002, Q4 Q_PMOS_GSD, Q5 BTA24-600CW, Q6 Q_NPN_BEC, Q7 Q_NPN_BEC, SW1 SW_SPDT_WITH_SHIELD, SW2 SW_SPDT_WITH_SHIELD, SW3 SW_PUSH_SMALL_H, SW4 SW_PUSH_SMALL_H, U1 PC817, U2 TPS53319, U3 CM1293A-04SO, U4 AZ1117-3.3, U5 AZ1117-5.0, U6 CH340G, U7 CM1293A-04SO, U8 ESP-WROOM-02, U9 TLP561J, Y1 Crystal

Commit message: Added a spark killer
Parts:
- Q5: footprint Package_TO_SOT_THT:TO-220-3_Horizontal_TabDown -> Package_TO_SOT_THT:TO-220-3_Vertical
Changed lines of the file:
@@
 U 1 1 5BFFD01E
 P 5800 1250
-F 0 "K1" H 6230 1296 50  0000 L CNN
-F 1 "953-1C-5DG-1" H 6230 1205 50  0000 L CNN
+F 0 "K1" H 5750 950 50  0000 L CNN
+F 1 "953-1C-5DG-1" H 5750 850 50  0000 L CNN
 F 2 "thisproject:953-1C-5DG-1" H 6250 1200 50  0001 L CNN
 F 3 "http://www.hsinda.com.cn/en/imgdown.asp?FileName=UploadFiles/201431310240386.pdf" H 5800 1250 50  0001 C CNN
@@
 F 0 "Q5" H 7328 2746 50  0000 L CNN
 F 1 "BTA24-600CW" H 7328 2655 50  0000 L CNN
-F 2 "Package_TO_SOT_THT:TO-220-3_Horizontal_TabDown" H 7400 2625 50  0001 L CIN
+F 2 "Package_TO_SOT_THT:TO-220-3_Vertical" H 7400 2625 50  0001 L CIN
 F 3 "http://pdf.datasheetcatalog.com/datasheet/PowerInnovations/mXuqxvy.pdf" H 7200 2700 50  0001 L CNN
 	1    7200 2700

Commit message: To make easy chassis making
Parts:
- added F14: 15A, components:FUSE-HOLDER-FUC-03A-20mm_x_5.2mm, symbol Device:Fuse_Small
- F3, F4: footprint Fuse:Fuse_Bourns_MF-RG800 -> Fuse:Fuse_Bourns_MF-RG700
- R26: footprint Resistor_THT:R_Axial_Power_L48.0mm_W12.5mm_P55.88mm -> Resistor_THT:R_Axial_Power_L25.0mm_W9.0mm_P27.94mm
- SW2: footprint components:SW_SPDT_WITH_SHILD -> components:SW_SPDT_v
Connections:
- net labels added: AC_OUT_L_2
- wire segments 559 -> 561
Changed lines of the file:
@@
 F 0 "F3" H 2318 5146 50  0000 L CNN
 F 1 "3A hold" H 2318 5055 50  0000 L CNN
-F 2 "Fuse:Fuse_Bourns_MF-RG800" H 2300 4900 50  0001 L CNN
+F 2 "Fuse:Fuse_Bourns_MF-RG700" H 2300 4900 50  0001 L CNN
 F 3 "" H 2250 5100 50  0001 C CNN
 	1    2250 5100
@@
 F 0 "SW2" H 2600 6265 50  0000 C CNN
 F 1 "SW_SPDT_WITH_SHIELD" H 2600 6174 50  0000 C CNN
-F 2 "components:SW_SPDT_WITH_SHILD" H 2600 5950 50  0001 C CNN
+F 2 "components:SW_SPDT_v" H 2600 5950 50  0001 C CNN
 F 3 "" H 2600 5950 50  0001 C CNN
 	1    2600 5950
@@
 F 0 "F4" H 2318 5246 50  0000 L CNN
 F 1 "3A hold" H 2318 5155 50  0000 L CNN
-F 2 "Fuse:Fuse_Bourns_MF-RG800" H 2300 5000 50  0001 L CNN
+F 2 "Fuse:Fuse_Bourns_MF-RG700" H 2300 5000 50  0001 L CNN
 F 3 "" H 2250 5200 50  0001 C CNN
 	1    2250 5200
@@
 F 0 "R26" V 7750 2050 50  0000 C CNN
 F 1 "100R" V 7850 2050 50  0000 C CNN
-F 2 "Resistor_THT:R_Axial_Power_L48.0mm_W12.5mm_P55.88mm" V 8063 2050 50  0001 C CNN
+F 2 "Resistor_THT:R_Axial_Power_L25.0mm_W9.0mm_P27.94mm" V 8063 2050 50  0001 C CNN
 F 3 "~" H 7950 2050 50  0001 C CNN
 	1    7950 2050
@@
 L Connector:Conn_WallPlug P1
 U 1 1 5C0508C7
-P 9050 900
-F 0 "P1" H 8840 946 50  0000 R CNN
-F 1 "Conn_WallPlug" H 8840 855 50  0000 R CNN
-F 2 "Connector_Wire:SolderWirePad_1x02_P7.62mm_Drill2mm" H 9450 900 50  0001 C CNN
-F 3 "~" H 9450 900 50  0001 C CNN
-	1    9050 900
+P 9450 900
+F 0 "P1" H 9240 946 50  0000 R CNN
+F 1 "Conn_WallPlug" H 9240 855 50  0000 R CNN
+F 2 "Connector_Wire:SolderWirePad_1x02_P7.62mm_Drill2mm" H 9850 900 50  0001 C CNN
+F 3 "~" H 9850 900 50  0001 C CNN
+	1    9450 900
 	-1   0    0    -1
 $EndComp
@@
 L Connector:Conn_WallSocket J6
 U 1 1 5C05103E
-P 9050 1650
-F 0 "J6" H 9204 1696 50  0000 L CNN
-F 1 "Conn_WallSocket" H 9204 1605 50  0000 L CNN
-F 2 "Connector_Wire:SolderWirePad_1x02_P7.62mm_Drill2mm" H 8650 1650 50  0001 C CNN
-F 3 "~" H 8650 1650 50  0001 C CNN
-	1    9050 1650
+P 9450 1650
+F 0 "J6" H 9604 1696 50  0000 L CNN
+F 1 "Conn_WallSocket" H 9604 1605 50  0000 L CNN
+F 2 "Connector_Wire:SolderWirePad_1x02_P7.62mm_Drill2mm" H 9050 1650 50  0001 C CNN
+F 3 "~" H 9050 1650 50  0001 C CNN
+	1    9450 1650
 	1    0    0    -1
 $EndComp
@@
 $EndComp
 Wire Wire Line
-	8850 800  8250 800
-Wire Wire Line
 	8250 800  8250 850
 Wire Wire Line
-	8850 1000 8250 1000
-Wire Wire Line
 	8250 1000 8250 950
 $Comp
@@
 	8100 2050 9100 2050
 Wire Wire Line
-	8850 1750 8250 1750
-Wire Wire Line
 	8250 1750 8250 1000
 Connection ~ 8250 1000
@@
 Wire Wire Line
 	6500 1550 7000 1550
+$Comp
+L Device:Fuse_Small F14
+U 1 1 5C1B838A
+P 9050 1550
+F 0 "F14" H 9050 1735 50  0000 C CNN
+F 1 "15A" H 9050 1644 50  0000 C CNN
+F 2 "components:FUSE-HOLDER-FUC-03A-20mm_x_5.2mm" H 9050 1550 50  0001 C CNN
+F 3 "~" H 9050 1550 50  0001 C CNN
+	1    9050 1550
+	1    0    0    -1
+$EndComp
+Wire Wire Line
+	8250 1000 9250 1000
+Wire Wire Line
+	8250 800  9250 800
+Wire Wire Line
+	8950 1550 8850 1550
+Wire Wire Line
+	9150 1550 9250 1550
+Wire Wire Line
+	8250 1750 9250 1750
+Text Label 9200 1550 1    50   ~ 0
+AC_OUT_L_2
 $EndSCHEMATC
